File: pcb/Lucky15.kicad_pcb (KiCad board)
At the start: 2 copper layers, 81 x 98.8 mm, 36 parts, among them J1 OLED_128x32, SW8 RotaryEncoder_Switch, U1 ProMicro

Commit message: Update PCB Uploads to current version with power switch
Parts:
- added SW1: SW_SPDT, Button_Switch_SMD:SW_SPDT_Shouhan_MSK12C02, F.Cu at (154.8, 44.2)
Connections:
- BT1 pad 1: BATT+ -> Net-(BT1-+)
Routing:
- net Net-(BT1-+): track 0.00 -> 19.4 mm, vias 0 -> 1
- net BATT-: track 70.7 -> 78.8 mm
- net BATT+: track 74.7 -> 69.9 mm, vias 4 -> 0
