File: pcb/Lucky15.kicad_sch (KiCad schematic)
At the start: 35 parts, among them J1 OLED_128x32, SW8 RotaryEncoder_Switch, U1 ProMicro

Commit message: Update PCB Uploads to current version with power switch
Parts:
- added SW1: SW_SPDT, Button_Switch_SMD:SW_SPDT_Shouhan_MSK12C02, symbol Switch:SW_SPDT
Connections:
- net BATT+: now also SW1.1 (A); no longer BT1.1 (+)
- new net: BT1.1 (+), SW1.2 (B)
Other:
- moved on the sheet: BT1
Changed lines of the file:
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@@
 	(global_label "BATT-"
 		(shape input)
-		(at 185.42 73.66 0)
+		(at 189.23 74.93 0)
 		(fields_autoplaced yes)
 		(effects
@@
 		)
 		(property "Intersheetrefs" "${INTERSHEET_REFS}"
-			(at 194.2714 73.66 0)
+			(at 198.0814 74.93 0)
 			(hide yes)
 			(show_name no)
@@
 	(global_label "BATT+"
 		(shape input)
-		(at 175.26 73.66 180)
+		(at 168.91 77.47 180)
 		(fields_autoplaced yes)
 		(effects
@@
 		)
 		(property "Intersheetrefs" "${INTERSHEET_REFS}"
-			(at 166.4086 73.66 0)
+			(at 160.0586 77.47 0)
 			(hide yes)
 			(show_name no)
@@
 	)
 	(symbol
+		(lib_id "Switch:SW_SPDT")
+		(at 173.99 74.93 180)
+		(unit 1)
+		(body_style 1)
+		(exclude_from_sim no)
+		(in_bom yes)
+		(on_board yes)
+		(in_pos_files yes)
+		(dnp no)
+		(fields_autoplaced yes)
+		(property "Reference" "SW1"
+			(at 173.99 66.04 0)
+			(show_name no)
+			(do_not_autoplace no)
+			(effects
+				(font
+					(size 1.27 1.27)
+				)
+			)
+		)
+		(property "Value" "SW_SPDT"
+			(at 173.99 68.58 0)
+			(show_name no)
+			(do_not_autoplace no)
+			(effects
+				(font
+					(size 1.27 1.27)
+				)
+			)
+		)
+		(property "Footprint" "Button_Switch_SMD:SW_SPDT_Shouhan_MSK12C02"
+			(at 173.99 74.93 0)
+			(hide yes)
+			(show_name no)
+			(do_not_autoplace no)
+			(effects
+				(font
+					(size 1.27 1.27)
+				)
+			)
+		)
+		(property "Datasheet" ""
+			(at 173.99 67.31 0)
+			(hide yes)
+			(show_name no)
+			(do_not_autoplace no)
+			(effects
+				(font
+					(size 1.27 1.27)
+				)
+			)
+		)
+		(property "Description" "Switch, single pole double throw"
+			(at 173.99 74.93 0)
+			(hide yes)
+			(show_name no)
+			(do_not_autoplace no)
+			(effects
+				(font
+					(size 1.27 1.27)
+				)
+			)
+		)
+		(pin "3"
+		)
+		(pin "1"
+		)
+		(pin "2"
+		)
+		(instances
+			(project "Lucky15"
+				(path "/d6a2b069-1da0-4ba9-b086-6a1c47b64c3b"
+					(reference "SW1")
+					(unit 1)
+				)
+			)
+		)
+	)
+	(symbol
 		(lib_id "ScottoKeebs:Placeholder_Diode")
 		(at 116.84 106.68 0)
@@
 	(symbol
 		(lib_id "Device:Battery")
-		(at 180.34 73.66 90)
+		(at 184.15 74.93 90)
 		(unit 1)
 		(body_style 1)
@@
 		(fields_autoplaced yes)
 		(property "Reference" "BT1"
-			(at 178.4984 69.85 0)
+			(at 182.3084 71.12 0)
 			(show_name no)
 			(do_not_autoplace no)
@@
 		)
 		(property "Value" "Battery"
-			(at 181.0384 69.85 0)
+			(at 184.8484 71.12 0)
 			(show_name no)
 			(do_not_autoplace no)
@@
 		)
 		(property "Footprint" "Connector_JST:JST_PH_S2B-PH-SM4-TB_1x02-1MP_P2.00mm_Horizontal"
-			(at 178.816 73.66 90)
+			(at 182.626 74.93 90)
 			(hide yes)
 			(show_name no)
@@
 		)
 		(property "Datasheet" ""
-			(at 178.816 73.66 90)
+			(at 182.626 74.93 90)
 			(hide yes)
 			(show_name no)
@@
 		)
 		(property "Description" "Multiple-cell battery"
-			(at 180.34 73.66 0)
+			(at 184.15 74.93 0)
 			(hide yes)
 			(show_name no)
@@
 		)
 		(property "Sim.Device" "V"
-			(at 180.34 73.66 0)
+			(at 184.15 74.93 0)
 			(hide yes)
 			(show_name no)
@@
 		)
 		(property "Sim.Type" "DC"
-			(at 180.34 73.66 0)
+			(at 184.15 74.93 0)
 			(hide yes)
 			(show_name no)
@@
 		)
 		(property "Sim.Pins" "1=+ 2=-"
-			(at 180.34 73.66 0)
-			(hide yes)
-			(show_name no)
+			(at 184.15 74.93 0)
+			(hide yes)
+			(show_name no)
